File: hardware/whypod.sch (EAGLE design)
At the start: 13 parts, among them IC1 IC_USBLC6-2, X2 USB-A-S, Y1 CRYSTAL-GROUNDEDSMD-5X3.2

Commit message: Hardware updates
Parts:
- removed R3: 0R, rcl:R-EU_R0603
- added C6, C7, C8, C9: (no value), rcl:C-EUC0603
Connections:
- removed net N$5: R3.1, U$2.PD7
- new net LCD_BACKLIGHT: U$2.PC6
- new net SDIO_CLK: U$2.PC12
- new net SDIO_CMD: U$2.PD2
- new net SDIO_D0: U$2.PC8
- new net SDIO_D1: U$2.PC9
- new net SDIO_D2: U$2.PC10
- new net SDIO_D3: U$2.PC11
- net 3V: now also C6.1, C7.1, C8.1, C9.1
- net GND: now also C6.2, C7.2, C8.2, C9.2
- net LCD_CS: now also U$2.PD7; no longer R3.2
Changed lines of the file:
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@@
 <part name="GND2" library="supply1" deviceset="GND" device=""/>
 <part name="GND3" library="supply1" deviceset="GND" device=""/>
-<part name="R3" library="rcl" deviceset="R-EU_" device="R0603" value="0R"/>
 <part name="C1" library="rcl" deviceset="C-EU" device="C0603" value="22 pF"/>
 <part name="C2" library="rcl" deviceset="C-EU" device="C0603" value="22 pF"/>
@@
 <part name="IC1" library="dp_devices" deviceset="IC_USBLC6-2" device=""/>
 <part name="GND10" library="supply1" deviceset="GND" device=""/>
+<part name="C6" library="rcl" deviceset="C-EU" device="C0603"/>
+<part name="GND11" library="supply1" deviceset="GND" device=""/>
+<part name="C7" library="rcl" deviceset="C-EU" device="C0603"/>
+<part name="GND12" library="supply1" deviceset="GND" device=""/>
+<part name="C8" library="rcl" deviceset="C-EU" device="C0603"/>
+<part name="GND13" library="supply1" deviceset="GND" device=""/>
+<part name="C9" library="rcl" deviceset="C-EU" device="C0603"/>
+<part name="GND14" library="supply1" deviceset="GND" device=""/>
 </parts>
 <sheets>
@@
 <instance part="GND2" gate="1" x="201.93" y="-45.72"/>
 <instance part="GND3" gate="1" x="213.36" y="-45.72"/>
-<instance part="R3" gate="G$1" x="269.24" y="2.54"/>
 <instance part="C1" gate="G$1" x="180.34" y="132.08"/>
 <instance part="C2" gate="G$1" x="172.72" y="132.08"/>
@@
 <instance part="IC1" gate="G$1" x="264.16" y="152.4" rot="R180"/>
 <instance part="GND10" gate="1" x="289.56" y="134.62"/>
+<instance part="C6" gate="G$1" x="177.292" y="213.36"/>
+<instance part="GND11" gate="1" x="177.292" y="203.2"/>
+<instance part="C7" gate="G$1" x="184.912" y="213.36"/>
+<instance part="GND12" gate="1" x="184.912" y="203.2"/>
+<instance part="C8" gate="G$1" x="192.532" y="213.36"/>
+<instance part="GND13" gate="1" x="192.532" y="203.2"/>
+<instance part="C9" gate="G$1" x="200.152" y="213.36"/>
+<instance part="GND14" gate="1" x="200.152" y="203.2"/>
 </instances>
 <busses>
@@
 <wire x1="289.56" y1="144.78" x2="289.56" y2="137.16" width="0.1524" layer="91"/>
 </segment>
+<segment>
+<pinref part="C6" gate="G$1" pin="2"/>
+<pinref part="GND11" gate="1" pin="GND"/>
+<wire x1="177.292" y1="205.74" x2="177.292" y2="208.28" width="0.1524" layer="91"/>
+</segment>
+<segment>
+<pinref part="C7" gate="G$1" pin="2"/>
+<pinref part="GND12" gate="1" pin="GND"/>
+<wire x1="184.912" y1="205.74" x2="184.912" y2="208.28" width="0.1524" layer="91"/>
+</segment>
+<segment>
+<pinref part="C8" gate="G$1" pin="2"/>
+<pinref part="GND13" gate="1" pin="GND"/>
+<wire x1="192.532" y1="205.74" x2="192.532" y2="208.28" width="0.1524" layer="91"/>
+</segment>
+<segment>
+<pinref part="C9" gate="G$1" pin="2"/>
+<pinref part="GND14" gate="1" pin="GND"/>
+<wire x1="200.152" y1="205.74" x2="200.152" y2="208.28" width="0.1524" layer="91"/>
+</segment>
 </net>
 <net name="DB0" class="0">
@@
 </segment>
 <segment>
+<label x="279.4" y="20.32" size="1.4224" layer="95" xref="yes"/>
 <pinref part="U$2" gate="G$1" pin="PD0"/>
-<wire x1="246.38" y1="20.32" x2="256.54" y2="20.32" width="0.1524" layer="91"/>
-<label x="256.54" y="20.32" size="1.4224" layer="95" xref="yes"/>
+<wire x1="279.4" y1="20.32" x2="246.38" y2="20.32" width="0.1524" layer="91"/>
 </segment>
 </net>
@@
 </segment>
 <segment>
-<pinref part="R3" gate="G$1" pin="2"/>
-<wire x1="274.32" y1="2.54" x2="279.4" y2="2.54" width="0.1524" layer="91"/>
 <label x="279.4" y="2.54" size="1.4224" layer="95" xref="yes"/>
+<pinref part="U$2" gate="G$1" pin="PD7"/>
+<wire x1="246.38" y1="2.54" x2="279.4" y2="2.54" width="0.1524" layer="91"/>
 </segment>
 </net>
@@
 <wire x1="246.38" y1="-10.16" x2="256.54" y2="-10.16" width="0.1524" layer="91"/>
 <label x="256.54" y="-10.16" size="1.4224" layer="95" xref="yes"/>
-</segment>
-</net>
-<net name="N$5" class="0">
-<segment>
-<pinref part="U$2" gate="G$1" pin="PD7"/>
-<pinref part="R3" gate="G$1" pin="1"/>
-<wire x1="264.16" y1="2.54" x2="246.38" y2="2.54" width="0.1524" layer="91"/>
 </segment>
 </net>
@@
 <wire x1="165.1" y1="218.44" x2="169.672" y2="218.44" width="0.1524" layer="91"/>
 <pinref part="C5" gate="G$1" pin="1"/>
-<wire x1="169.672" y1="218.44" x2="182.88" y2="218.44" width="0.1524" layer="91"/>
+<wire x1="169.672" y1="218.44" x2="177.292" y2="218.44" width="0.1524" layer="91"/>
+<wire x1="177.292" y1="218.44" x2="184.912" y2="218.44" width="0.1524" layer="91"/>
+<wire x1="184.912" y1="218.44" x2="192.532" y2="218.44" width="0.1524" layer="91"/>
+<wire x1="192.532" y1="218.44" x2="200.152" y2="218.44" width="0.1524" layer="91"/>
+<wire x1="200.152" y1="218.44" x2="223.52" y2="218.44" width="0.1524" layer="91"/>
 <wire x1="169.672" y1="215.9" x2="169.672" y2="218.44" width="0.1524" layer="91"/>
 <junction x="169.672" y="218.44"/>
+<pinref part="C6" gate="G$1" pin="1"/>
+<wire x1="177.292" y1="215.9" x2="177.292" y2="218.44" width="0.1524" layer="91"/>
+<junction x="177.292" y="218.44"/>
+<pinref part="C7" gate="G$1" pin="1"/>
+<wire x1="184.912" y1="215.9" x2="184.912" y2="218.44" width="0.1524" layer="91"/>
+<junction x="184.912" y="218.44"/>
+<pinref part="C8" gate="G$1" pin="1"/>
+<wire x1="192.532" y1="215.9" x2="192.532" y2="218.44" width="0.1524" layer="91"/>
+<junction x="192.532" y="218.44"/>
+<pinref part="C9" gate="G$1" pin="1"/>
+<wire x1="200.152" y1="215.9" x2="200.152" y2="218.44" width="0.1524" layer="91"/>
+<junction x="200.152" y="218.44"/>
 </segment>
 </net>
@@
 </segment>
 </net>
+<net name="LCD_BACKLIGHT" class="0">
+<segment>
+<pinref part="U$2" gate="G$1" pin="PC6"/>
+<wire x1="246.38" y1="48.26" x2="256.54" y2="48.26" width="0.1524" layer="91"/>
+<label x="256.54" y="48.26" size="1.4224" layer="95" xref="yes"/>
+</segment>
+</net>
+<net name="SDIO_D0" class="0">
+<segment>
+<pinref part="U$2" gate="G$1" pin="PC8"/>
+<wire x1="246.38" y1="43.18" x2="256.54" y2="43.18" width="0.1524" layer="91"/>
+<label x="256.54" y="43.18" size="1.4224" layer="95" xref="yes"/>
+</segment>
+</net>
+<net name="SDIO_D1" class="0">
+<segment>
+<pinref part="U$2" gate="G$1" pin="PC9"/>
+<wire x1="246.38" y1="40.64" x2="256.54" y2="40.64" width="0.1524" layer="91"/>
+<label x="256.54" y="40.64" size="1.4224" layer="95" xref="yes"/>
+</segment>
+</net>
+<net name="SDIO_D2" class="0">
+<segment>
+<pinref part="U$2" gate="G$1" pin="PC10"/>
+<wire x1="246.38" y1="38.1" x2="256.54" y2="38.1" width="0.1524" layer="91"/>
+<label x="256.54" y="38.1" size="1.4224" layer="95" xref="yes"/>
+</segment>
+</net>
+<net name="SDIO_D3" class="0">
+<segment>
+<pinref part="U$2" gate="G$1" pin="PC11"/>
+<wire x1="246.38" y1="35.56" x2="256.54" y2="35.56" width="0.1524" layer="91"/>
+<label x="256.54" y="35.56" size="1.4224" layer="95" xref="yes"/>
+</segment>
+</net>
+<net name="SDIO_CLK" class="0">
+<segment>
+<pinref part="U$2" gate="G$1" pin="PC12"/>
+<wire x1="246.38" y1="33.02" x2="256.54" y2="33.02" width="0.1524" layer="91"/>
+<label x="256.54" y="33.02" size="1.4224" layer="95" xref="yes"/>
+</segment>
+</net>
+<net name="SDIO_CMD" class="0">
+<segment>
+<pinref part="U$2" gate="G$1" pin="PD2"/>
+<wire x1="246.38" y1="15.24" x2="256.54" y2="15.24" width="0.1524" layer="91"/>
+<label x="256.54" y="15.24" size="1.4224" layer="95" xref="yes"/>
+</segment>
+</net>

Commit message: Hardware updated
Parts:
- added C10: (no value), rcl:C-EUC0603
- added JP1: (no value), pinhead-2:PINHD-1X04_2.54-SMD-90°
- added R1, R2: 0R, rcl:R-EU_R0603
- added R10, R11, R3, R6, R8: (no value), rcl:R-EU_R0603
- added R7, R9: (no value), rcl:R-EU_R0402
- added U1: USD-SOCKETUSD, SparkFun-Connectors:USD-SOCKETUSD
Connections:
- new net N$5: R1.2, U$2.PC10
- new net N$8: R2.2, U$2.PC11
- new net SDIO_CD: R10.1, U$2.PD3, U1.SHIELD@1
- net 3V: now also C10.1, R10.2, R11.2, R3.2, R6.2, R7.2, R8.2, R9.2, U1.VCC
- net GND: now also C10.2, U1.GND, U1.SHIELD@2, U1.SHIELD@3, U1.SHIELD@4
- net SDIO_CLK: now also R9.1, U1.SCK
- net SDIO_CMD: now also R11.1, U1.DI
- net SDIO_D0: now also R3.1, U1.DO
- net SDIO_D1: now also R6.1, U1.RSV
- net SDIO_D2: now also R1.1, R7.1, U1.NC; no longer U$2.PC10
- net SDIO_D3: now also R2.1, R8.1, U1.CS; no longer U$2.PC11
- net SWD_CLK: now also JP1.4
- net SWD_IO: now also JP1.3

Commit message: PCB updates
Parts:
- removed JP1: (no value), pinhead-2:PINHD-1X04_2.54-SMD-90°
- added J1: AUDIO_JACK_TRRSSMD_RA, SparkFun-Connectors:AUDIO_JACK_TRRSSMD_RA
- added JP3: (no value), pinhead-2:PINHD-1X06_2.54-SMD-90°
- added U$1: WM8731, microdecv1:WM8731
Connections:
- new net NRST: JP3.5, U$2.NRST
- new net SWD_SWO: JP3.6
- net 3V: now also JP3.1
- net GND: now also JP3.3
- net SWD_CLK: now also JP3.2; no longer JP1.4
- net SWD_IO: now also JP3.4; no longer JP1.3
Changed lines of the file:
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@@
 <part name="R10" library="rcl" deviceset="R-EU_" device="R0603"/>
 <part name="R11" library="rcl" deviceset="R-EU_" device="R0603"/>
-<part name="JP1" library="pinhead-2" deviceset="PINHD-1X04" device="_2.54-SMD-90°"/>
+<part name="JP3" library="pinhead-2" deviceset="PINHD-1X06" device="_2.54-SMD-90°"/>
+<part name="GND17" library="supply1" deviceset="GND" device=""/>
+<part name="J1" library="SparkFun-Connectors" deviceset="AUDIO_JACK_TRRS" device="SMD_RA"/>
+<part name="U$1" library="microdecv1" deviceset="WM8731" device=""/>
 </parts>
 <sheets>
@@
 <instance part="R10" gate="G$1" x="365.76" y="167.64" rot="R90"/>
 <instance part="R11" gate="G$1" x="360.68" y="167.64" rot="R90"/>
-<instance part="JP1" gate="A" x="411.48" y="215.9"/>
+<instance part="JP3" gate="A" x="406.4" y="218.44"/>
+<instance part="GND17" gate="1" x="396.24" y="205.74"/>
+<instance part="J1" gate="G$1" x="393.7" y="259.08"/>
+<instance part="U$1" gate="G$1" x="340.36" y="271.78" rot="MR0"/>
 </instances>
 <busses>
@@
 <wire x1="207.772" y1="205.74" x2="207.772" y2="208.28" width="0.1524" layer="91"/>
 </segment>
+<segment>
+<pinref part="JP3" gate="A" pin="3"/>
+<wire x1="403.86" y1="220.98" x2="396.24" y2="220.98" width="0.1524" layer="91"/>
+<wire x1="396.24" y1="220.98" x2="396.24" y2="208.28" width="0.1524" layer="91"/>
+<pinref part="GND17" gate="1" pin="GND"/>
+</segment>
 </net>
 <net name="DB0" class="0">
@@
 </segment>
 <segment>
-<pinref part="JP1" gate="A" pin="3"/>
-<wire x1="408.94" y1="215.9" x2="396.24" y2="215.9" width="0.1524" layer="91"/>
+<wire x1="403.86" y1="218.44" x2="393.7" y2="218.44" width="0.1524" layer="91"/>
+<label x="393.7" y="218.44" size="1.4224" layer="95" rot="R180" xref="yes"/>
+<pinref part="JP3" gate="A" pin="4"/>
 </segment>
 </net>
@@
 </segment>
 <segment>
-<pinref part="JP1" gate="A" pin="4"/>
-<wire x1="408.94" y1="213.36" x2="396.24" y2="213.36" width="0.1524" layer="91"/>
+<wire x1="403.86" y1="223.52" x2="393.7" y2="223.52" width="0.1524" layer="91"/>
+<label x="393.7" y="223.52" size="1.4224" layer="95" rot="R180" xref="yes"/>
+<pinref part="JP3" gate="A" pin="2"/>
 </segment>
 </net>
@@
 <junction x="365.76" y="175.26"/>
 </segment>
+<segment>
+<pinref part="JP3" gate="A" pin="1"/>
+<wire x1="403.86" y1="226.06" x2="393.7" y2="226.06" width="0.1524" layer="91"/>
+</segment>
 </net>
 <net name="_5V" class="0">
@@
 </segment>
 </net>
+<net name="NRST" class="0">
+<segment>
+<pinref part="JP3" gate="A" pin="5"/>
+<wire x1="403.86" y1="215.9" x2="393.7" y2="215.9" width="0.1524" layer="91"/>
+<label x="393.7" y="215.9" size="1.4224" layer="95" rot="R180" xref="yes"/>
+</segment>
+<segment>
+<pinref part="U$2" gate="G$1" pin="NRST"/>
+<wire x1="177.8" y1="76.2" x2="177.8" y2="81.28" width="0.1524" layer="91"/>
+<label x="177.8" y="81.28" size="1.4224" layer="95" rot="R90" xref="yes"/>
+</segment>
+</net>
+<net name="SWD_SWO" class="0">
+<segment>
+<pinref part="JP3" gate="A" pin="6"/>
+<wire x1="403.86" y1="213.36" x2="393.7" y2="213.36" width="0.1524" layer="91"/>
+<label x="393.7" y="213.36" size="1.4224" layer="95" rot="R180" xref="yes"/>
+</segment>
+</net>

Commit message: PCB updated
Parts:
- removed JP3: (no value), pinhead-2:PINHD-1X06_2.54-SMD-90°
- added JP1: (no value), pinhead-2:PINHD-1X06_2.54-SMD-90°
Connections:
- new net AGND: J1.EARTH, U$1.AGND
- new net I2C1_SCL: U$1.SCLK, U$2.PB6
- new net I2C1_SDA: U$1.SDIN, U$2.PB7
- new net I2S_WS: U$2.PA15
- net 3V: now also JP1.1; no longer JP3.1
- net GND: now also JP1.3, U$1.DGND; no longer JP3.3
- net NRST: now also JP1.5; no longer JP3.5
- net SWD_CLK: now also JP1.2; no longer JP3.2
- net SWD_IO: now also JP1.4; no longer JP3.4
- net SWD_SWO: now also JP1.6; no longer JP3.6
Other:
- moved on the sheet: J1, U$1
Changed lines of the file:
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@@
 <part name="R10" library="rcl" deviceset="R-EU_" device="R0603"/>
 <part name="R11" library="rcl" deviceset="R-EU_" device="R0603"/>
-<part name="JP3" library="pinhead-2" deviceset="PINHD-1X06" device="_2.54-SMD-90°"/>
-<part name="GND17" library="supply1" deviceset="GND" device=""/>
 <part name="J1" library="SparkFun-Connectors" deviceset="AUDIO_JACK_TRRS" device="SMD_RA"/>
 <part name="U$1" library="microdecv1" deviceset="WM8731" device=""/>
+<part name="GND17" library="supply1" deviceset="GND" device=""/>
+<part name="JP1" library="pinhead-2" deviceset="PINHD-1X06" device="_2.54-SMD-90°"/>
 </parts>
 <sheets>
@@
 <instance part="R10" gate="G$1" x="365.76" y="167.64" rot="R90"/>
 <instance part="R11" gate="G$1" x="360.68" y="167.64" rot="R90"/>
-<instance part="JP3" gate="A" x="406.4" y="218.44"/>
-<instance part="GND17" gate="1" x="396.24" y="205.74"/>
-<instance part="J1" gate="G$1" x="393.7" y="259.08"/>
-<instance part="U$1" gate="G$1" x="340.36" y="271.78" rot="MR0"/>
+<instance part="J1" gate="G$1" x="401.32" y="261.62" rot="R180"/>
+<instance part="U$1" gate="G$1" x="332.74" y="271.78" rot="MR0"/>
+<instance part="GND17" gate="1" x="312.42" y="241.3"/>
+<instance part="JP1" gate="A" x="464.82" y="259.08"/>
 </instances>
 <busses>
@@
 </segment>
 <segment>
-<pinref part="JP3" gate="A" pin="3"/>
-<wire x1="403.86" y1="220.98" x2="396.24" y2="220.98" width="0.1524" layer="91"/>
-<wire x1="396.24" y1="220.98" x2="396.24" y2="208.28" width="0.1524" layer="91"/>
+<pinref part="U$1" gate="G$1" pin="DGND"/>
+<wire x1="314.96" y1="287.02" x2="312.42" y2="287.02" width="0.1524" layer="91"/>
+<wire x1="312.42" y1="287.02" x2="312.42" y2="243.84" width="0.1524" layer="91"/>
 <pinref part="GND17" gate="1" pin="GND"/>
+</segment>
+<segment>
+<pinref part="JP1" gate="A" pin="3"/>
+<wire x1="462.28" y1="261.62" x2="452.12" y2="261.62" width="0.1524" layer="91"/>
 </segment>
 </net>
@@
 </segment>
 <segment>
-<wire x1="403.86" y1="218.44" x2="393.7" y2="218.44" width="0.1524" layer="91"/>
-<label x="393.7" y="218.44" size="1.4224" layer="95" rot="R180" xref="yes"/>
-<pinref part="JP3" gate="A" pin="4"/>
+<pinref part="JP1" gate="A" pin="4"/>
+<wire x1="462.28" y1="259.08" x2="452.12" y2="259.08" width="0.1524" layer="91"/>
 </segment>
 </net>
@@
 </segment>
 <segment>
-<wire x1="403.86" y1="223.52" x2="393.7" y2="223.52" width="0.1524" layer="91"/>
-<label x="393.7" y="223.52" size="1.4224" layer="95" rot="R180" xref="yes"/>
-<pinref part="JP3" gate="A" pin="2"/>
+<pinref part="JP1" gate="A" pin="2"/>
+<wire x1="462.28" y1="264.16" x2="452.12" y2="264.16" width="0.1524" layer="91"/>
 </segment>
 </net>
@@
 </segment>
 <segment>
-<pinref part="JP3" gate="A" pin="1"/>
-<wire x1="403.86" y1="226.06" x2="393.7" y2="226.06" width="0.1524" layer="91"/>
+<pinref part="JP1" gate="A" pin="1"/>
+<wire x1="462.28" y1="266.7" x2="452.12" y2="266.7" width="0.1524" layer="91"/>
 </segment>
 </net>
@@
 <net name="NRST" class="0">
 <segment>
-<pinref part="JP3" gate="A" pin="5"/>
-<wire x1="403.86" y1="215.9" x2="393.7" y2="215.9" width="0.1524" layer="91"/>
-<label x="393.7" y="215.9" size="1.4224" layer="95" rot="R180" xref="yes"/>
-</segment>
-<segment>
 <pinref part="U$2" gate="G$1" pin="NRST"/>
 <wire x1="177.8" y1="76.2" x2="177.8" y2="81.28" width="0.1524" layer="91"/>
 <label x="177.8" y="81.28" size="1.4224" layer="95" rot="R90" xref="yes"/>
 </segment>
+<segment>
+<pinref part="JP1" gate="A" pin="5"/>
+<wire x1="462.28" y1="256.54" x2="452.12" y2="256.54" width="0.1524" layer="91"/>
+</segment>
+</net>
+<net name="AGND" class="0">
+<segment>
+<pinref part="J1" gate="G$1" pin="EARTH"/>
+<wire x1="396.24" y1="256.54" x2="388.62" y2="256.54" width="0.1524" layer="91"/>
+<label x="388.62" y="256.54" size="1.4224" layer="95" rot="R180" xref="yes"/>
+</segment>
+<segment>
+<pinref part="U$1" gate="G$1" pin="AGND"/>
+<wire x1="350.52" y1="289.56" x2="355.6" y2="289.56" width="0.1524" layer="91"/>
+<label x="355.6" y="289.56" size="1.4224" layer="95" xref="yes"/>
+</segment>
+</net>
+<net name="I2S_WS" class="0">
+<segment>
+<pinref part="U$2" gate="G$1" pin="PA15"/>
+<wire x1="158.75" y1="25.4" x2="152.4" y2="25.4" width="0.1524" layer="91"/>
+<label x="152.4" y="25.4" size="1.4224" layer="95" rot="R180" xref="yes"/>
+</segment>
+</net>
+<net name="I2C1_SCL" class="0">
+<segment>
+<pinref part="U$2" gate="G$1" pin="PB6"/>
+<wire x1="158.75" y1="5.08" x2="153.416" y2="5.08" width="0.1524" layer="91"/>
+<label x="153.416" y="5.08" size="1.4224" layer="95" rot="R180" xref="yes"/>
+</segment>
+<segment>
+<pinref part="U$1" gate="G$1" pin="SCLK"/>
+<wire x1="314.96" y1="271.78" x2="306.832" y2="271.78" width="0.1524" layer="91"/>
+<label x="306.832" y="271.78" size="1.4224" layer="95" rot="R180" xref="yes"/>
+</segment>
+</net>
+<net name="I2C1_SDA" class="0">
+<segment>
+<pinref part="U$2" gate="G$1" pin="PB7"/>
+<wire x1="158.75" y1="2.54" x2="153.416" y2="2.54" width="0.1524" layer="91"/>
+<label x="153.416" y="2.54" size="1.4224" layer="95" rot="R180" xref="yes"/>
+</segment>
+<segment>
+<pinref part="U$1" gate="G$1" pin="SDIN"/>
+<wire x1="314.96" y1="269.24" x2="306.832" y2="269.24" width="0.1524" layer="91"/>
+<label x="306.832" y="269.24" size="1.4224" layer="95" rot="R180" xref="yes"/>
+</segment>
 </net>
 <net name="SWD_SWO" class="0">
 <segment>
-<pinref part="JP3" gate="A" pin="6"/>
-<wire x1="403.86" y1="213.36" x2="393.7" y2="213.36" width="0.1524" layer="91"/>
-<label x="393.7" y="213.36" size="1.4224" layer="95" rot="R180" xref="yes"/>
-</segment>
-</net>
+<pinref part="JP1" gate="A" pin="6"/>
+<wire x1="462.28" y1="254" x2="452.12" y2="254" width="0.1524" layer="91"/>
+</segment>
+</net>

Commit message: DAC added
Parts:
- added C11, C12: 22 pF, rcl:C-EUC0603
- added C13, C16, C18, C19, C20: (no value), rcl:C-EUC0603
- added C14, C15, C17, C21, C22: (no value), rcl:CPOL-EUSMCA
- added C23, C24: (no value), rcl:CPOL-EUSMCE
- added C25: 1u, rcl:C-EUC0603
- added C26: 220p, rcl:C-EUC0603
- added JP5: USB_MICROB_PLUGCONN-11752, SparkFun-Connectors:USB_MICROB_PLUGCONN-11752
- added L1: (no value), rcl:L-EUL3225M
- added R12, R15: (no value), rcl:R-EU_R0603
- added R13, R14: 0R, rcl:R-EU_R0603
- added R16: (no value), rcl:R-EU_R0402
- added R17, R18, R25: 47k, rcl:R-EU_R0603
- added R26: 680, rcl:R-EU_R0603
- added T1: BC557, transistor-pnp:BC557
- added Y2: CRYSTAL-GROUNDEDSMD-5X3.2, SparkFun-Clocks:CRYSTAL-GROUNDEDSMD-5X3.2
Connections:
- removed net VCC: JP2.3
- new net A_3V: C15.+, C16.1, C17.+, C18.1, L1.2, U$1.AVDD, U$1.HPVDD
- new net I2S_CK: U$1.BCLK, U$2.PB3
- new net I2S_EXT_SD: U$1.ADCDAT, U$2.PB4
- new net I2S_SD: R13.2, U$1.DACDAT
- new net LOUT: C23.+, U$1.LHPOUT
- new net MICBIAS: R26.2, U$1.MICBIAS
- new net MICIN: C25.2, U$1.MICIN
- new net N$11: R12.1, T1.B
- new net N$12: C13.1, C14.+, U$1.VMID
- new net N$13: C23.-, J1.TIP, R17.2
- new net N$14: R13.1, U$2.PB5
- new net N$15: C24.-, J1.RING1, R18.2
- new net N$16: R14.1, R16.1, U$2.PB7
- new net N$55: C25.1, C26.2, J1.RING2, R25.2, R26.1
- new net ROUT: C24.+, U$1.RHPOUT
- new net XTI: C11.1, U$1.XTI/MCLK, Y2.1
- new net XTO: C12.1, U$1.XTO, Y2.2
- net 3V: now also C19.1, C20.1, C21.+, C22.+, JP2.3, L1.1, R15.2, R16.2, T1.E, U$1.DBVDD, U$1.DCVDD
- net AGND: now also C13.2, C14.-, C15.-, C16.2, C17.-, C18.2, C26.1, R17.1, R18.1, R25.1, U$1.HPGND
- net GND: now also C11.2, C12.2, C19.2, C20.2, C21.-, C22.-, JP5.GND, U$1.CSB, U$1.MODE, Y2.3
- net I2C1_SCL: now also R15.1
- net I2C1_SDA: now also R14.2; no longer U$2.PB7
- net I2S_WS: now also U$1.ADCLRC, U$1.DACLRC
- net LCD_BACKLIGHT: now also R12.2
- net LED_A: now also T1.C
Other:
- moved on the sheet: C10, C5, C6, C7, C8, C9, J1, JP1
