File: hardware/whypod.sch (EAGLE design)
At the start: 72 parts, among them IC1 IC_USBLC6-2, J1 AUDIO_JACK_TRRSSMD_RA, U1 USD-SOCKETUSD, X2 USB-A-S, Y1 CRYSTAL-GROUNDEDSMD-5X3.2, Y2 CRYSTAL-GROUNDEDSMD-5X3.2

Commit message: Power circuit updated
Parts:
- added C32: (no value), rcl:C-EUC0603
- added C33: (no value), rcl:CPOL-EUSMCC
- added L3: COILCRAFT-LPS4018, passives:COILCRAFT-LPS4018
- added R22, R23: 0R, rcl:R-EU_R0603
Connections:
- removed net N$23: U$5.EN, U$5.IN
- removed net VBAT: C27.1, U$3.VBAT
- new net ENUSB_CPU: R22.2, U$2.PC7
- new net LIPOL: C27.1, C32.1, L3.1, U$3.VBAT, U$5.EN, U$5.IN
- new net N$24: L3.2, U$5.SW
- new net USBFAULT_CPU: R23.2, U$2.PA8
- net 3V: now also C33.+
- net ENUSB: now also R22.1, U$5.!FAULT; no longer U$2.PC7, U$5.ENUSB
- net GND: now also C32.2, C33.-
- net USBFAULT: now also R23.1, U$5.ENUSB; no longer U$2.PA8, U$5.!FAULT
Changed lines of the file:
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@@
 <part name="R21" library="rcl" deviceset="R-EU_" device="R0603"/>
 <part name="GND36" library="supply1" deviceset="GND" device=""/>
+<part name="C32" library="rcl" deviceset="C-EU" device="C0603"/>
+<part name="GND37" library="supply1" deviceset="GND" device=""/>
+<part name="L3" library="passives" deviceset="COILCRAFT-LPS4018" device=""/>
+<part name="C33" library="rcl" deviceset="CPOL-EU" device="SMCC"/>
+<part name="GND38" library="supply1" deviceset="GND" device=""/>
+<part name="R22" library="rcl" deviceset="R-EU_" device="R0603" value="0R"/>
+<part name="R23" library="rcl" deviceset="R-EU_" device="R0603" value="0R"/>
 </parts>
 <sheets>
@@
 <instance part="R21" gate="G$1" x="378.46" y="411.48" rot="R90"/>
 <instance part="GND36" gate="1" x="378.46" y="401.32"/>
+<instance part="C32" gate="G$1" x="309.88" y="419.1"/>
+<instance part="GND37" gate="1" x="309.88" y="408.94"/>
+<instance part="L3" gate="G$1" x="322.58" y="429.26" rot="R90"/>
+<instance part="C33" gate="G$1" x="259.08" y="350.52"/>
+<instance part="GND38" gate="1" x="259.08" y="340.36"/>
+<instance part="R22" gate="G$1" x="381" y="436.88" rot="R90"/>
+<instance part="R23" gate="G$1" x="388.62" y="436.88" rot="R90"/>
 </instances>
 <busses>
@@
 <pinref part="GND36" gate="1" pin="GND"/>
 <wire x1="378.46" y1="403.86" x2="378.46" y2="406.4" width="0.1524" layer="91"/>
+</segment>
+<segment>
+<pinref part="C32" gate="G$1" pin="2"/>
+<pinref part="GND37" gate="1" pin="GND"/>
+<wire x1="309.88" y1="411.48" x2="309.88" y2="414.02" width="0.1524" layer="91"/>
+</segment>
+<segment>
+<pinref part="C33" gate="G$1" pin="-"/>
+<pinref part="GND38" gate="1" pin="GND"/>
+<wire x1="259.08" y1="342.9" x2="259.08" y2="345.44" width="0.1524" layer="91"/>
 </segment>
 </net>
@@
 </segment>
 <segment>
-<wire x1="266.7" y1="355.6" x2="271.272" y2="355.6" width="0.1524" layer="91"/>
+<wire x1="254" y1="355.6" x2="259.08" y2="355.6" width="0.1524" layer="91"/>
 <pinref part="C5" gate="G$1" pin="1"/>
+<wire x1="259.08" y1="355.6" x2="271.272" y2="355.6" width="0.1524" layer="91"/>
 <wire x1="271.272" y1="355.6" x2="278.892" y2="355.6" width="0.1524" layer="91"/>
 <wire x1="278.892" y1="355.6" x2="286.512" y2="355.6" width="0.1524" layer="91"/>
@@
 <wire x1="344.932" y1="353.06" x2="344.932" y2="355.6" width="0.1524" layer="91"/>
 <junction x="344.932" y="355.6"/>
+<pinref part="C33" gate="G$1" pin="+"/>
+<wire x1="259.08" y1="353.06" x2="259.08" y2="355.6" width="0.1524" layer="91"/>
+<junction x="259.08" y="355.6"/>
 </segment>
 <segment>
@@
 </segment>
 </net>
-<net name="VBAT" class="0">
+<net name="LIPOL" class="0">
 <segment>
 <pinref part="U$3" gate="G$1" pin="VBAT"/>
@@
 <junction x="116.84" y="355.6"/>
 </segment>
+<segment>
+<pinref part="U$5" gate="G$1" pin="EN"/>
+<wire x1="335.28" y1="421.64" x2="330.2" y2="421.64" width="0.1524" layer="91"/>
+<pinref part="U$5" gate="G$1" pin="IN"/>
+<wire x1="335.28" y1="424.18" x2="330.2" y2="424.18" width="0.1524" layer="91"/>
+<wire x1="330.2" y1="424.18" x2="330.2" y2="421.64" width="0.1524" layer="91"/>
+<wire x1="330.2" y1="424.18" x2="309.88" y2="424.18" width="0.1524" layer="91"/>
+<junction x="330.2" y="424.18"/>
+<wire x1="309.88" y1="424.18" x2="307.34" y2="424.18" width="0.1524" layer="91"/>
+<wire x1="314.96" y1="429.26" x2="309.88" y2="429.26" width="0.1524" layer="91"/>
+<wire x1="309.88" y1="429.26" x2="309.88" y2="424.18" width="0.1524" layer="91"/>
+<junction x="309.88" y="424.18"/>
+<pinref part="C32" gate="G$1" pin="1"/>
+<wire x1="309.88" y1="421.64" x2="309.88" y2="424.18" width="0.1524" layer="91"/>
+<pinref part="L3" gate="G$1" pin="1"/>
+</segment>
 </net>
 <net name="N$19" class="0">
@@
 <wire x1="104.14" y1="381" x2="104.14" y2="383.54" width="0.1524" layer="91"/>
 <pinref part="LED1" gate="G$1" pin="C"/>
-<wire x1="91.44" y1="383.54" x2="104.14" y2="383.54" width="0.1524" layer="91"/>
+<wire x1="104.14" y1="383.54" x2="91.44" y2="383.54" width="0.1524" layer="91"/>
 </segment>
 </net>
@@
 </segment>
 </net>
-<net name="N$23" class="0">
-<segment>
-<pinref part="U$5" gate="G$1" pin="EN"/>
-<wire x1="335.28" y1="421.64" x2="330.2" y2="421.64" width="0.1524" layer="91"/>
-<pinref part="U$5" gate="G$1" pin="IN"/>
-<wire x1="335.28" y1="424.18" x2="330.2" y2="424.18" width="0.1524" layer="91"/>
-<wire x1="330.2" y1="424.18" x2="330.2" y2="421.64" width="0.1524" layer="91"/>
-</segment>
-</net>
 <net name="ENUSB" class="0">
-<segment>
-<pinref part="U$5" gate="G$1" pin="ENUSB"/>
-<wire x1="375.92" y1="421.64" x2="381" y2="421.64" width="0.1524" layer="91"/>
-<label x="381" y="421.64" size="1.4224" layer="95" xref="yes"/>
-</segment>
-<segment>
-<pinref part="U$2" gate="G$1" pin="PC7"/>
-<wire x1="246.38" y1="45.72" x2="256.54" y2="45.72" width="0.1524" layer="91"/>
-<label x="256.54" y="45.72" size="1.4224" layer="95" xref="yes"/>
-</segment>
-</net>
-<net name="USBFAULT" class="0">
-<segment>
-<pinref part="U$2" gate="G$1" pin="PA8"/>
-<wire x1="158.75" y1="43.18" x2="152.4" y2="43.18" width="0.1524" layer="91"/>
-<label x="152.4" y="43.18" size="1.4224" layer="95" rot="R180" xref="yes"/>
-</segment>
 <segment>
 <pinref part="U$5" gate="G$1" pin="!FAULT"/>
 <wire x1="375.92" y1="424.18" x2="381" y2="424.18" width="0.1524" layer="91"/>
 <label x="381" y="424.18" size="1.4224" layer="95" xref="yes"/>
+<pinref part="R22" gate="G$1" pin="1"/>
+<wire x1="381" y1="431.8" x2="381" y2="424.18" width="0.1524" layer="91"/>
+</segment>
+</net>
+<net name="USBFAULT" class="0">
+<segment>
+<pinref part="U$5" gate="G$1" pin="ENUSB"/>
+<label x="381" y="421.64" size="1.4224" layer="95" xref="yes"/>
+<pinref part="R23" gate="G$1" pin="1"/>
+<wire x1="375.92" y1="421.64" x2="388.62" y2="421.64" width="0.1524" layer="91"/>
+<wire x1="388.62" y1="421.64" x2="388.62" y2="431.8" width="0.1524" layer="91"/>
 </segment>
 </net>
@@
 </segment>
 </net>
+<net name="N$24" class="0">
+<segment>
+<pinref part="U$5" gate="G$1" pin="SW"/>
+<wire x1="335.28" y1="429.26" x2="330.2" y2="429.26" width="0.1524" layer="91"/>
+<pinref part="L3" gate="G$1" pin="2"/>
+</segment>
+</net>
+<net name="ENUSB_CPU" class="0">
+<segment>
+<pinref part="R22" gate="G$1" pin="2"/>
+<wire x1="381" y1="441.96" x2="381" y2="444.5" width="0.1524" layer="91"/>
+</segment>
+<segment>
+<pinref part="U$2" gate="G$1" pin="PC7"/>
+<wire x1="246.38" y1="45.72" x2="256.54" y2="45.72" width="0.1524" layer="91"/>
+<label x="256.54" y="45.72" size="1.4224" layer="95" xref="yes"/>
+</segment>
+</net>
+<net name="USBFAULT_CPU" class="0">
+<segment>
+<pinref part="R23" gate="G$1" pin="2"/>
+<wire x1="388.62" y1="441.96" x2="388.62" y2="444.5" width="0.1524" layer="91"/>
+</segment>
+<segment>
+<pinref part="U$2" gate="G$1" pin="PA8"/>
+<wire x1="158.75" y1="43.18" x2="152.4" y2="43.18" width="0.1524" layer="91"/>
+<label x="152.4" y="43.18" size="1.4224" layer="95" rot="R180" xref="yes"/>
+</segment>
+</net>

Commit message: PCB updated
Parts:
- added C34, C35, C36, C37: (no value), rcl:C-EUC0805
- added C38: (no value), rcl:C-EUC0603
- added C39, R24, R27: (no value), rcl:R-EU_R0402
- added U$6: TPS63060, mw:TPS63060
- C33: device rcl:CPOL-EUSMCC -> rcl:C-EUC0805
- R12: device rcl:R-EU_R0603 -> rcl:R-EU_R0402
Connections:
- new net N$23: C38.1, U$6.VAUX
- new net N$25: C39.1, R24.2, R27.1, U$6.FB
- new net POWER_EN: U$2.PC6, U$6.EN
- net 3V: now also C33.1, C34.1, C35.1, R27.2, U$6.VOUT; no longer C33.+
- net GND: now also C33.2, C34.2, C35.2, C36.2, C37.2, C38.2, C39.2, R24.1, U$6.GND, U$6.PS/SYNC, U$6.TERM; no longer C33.-
- net LCD_BACKLIGHT: now also U$2.PB10; no longer U$2.PC6
- net LIPOL: now also C36.1, C37.1, U$6.VIN
Other:
- moved on the sheet: C27, C28, F3, JP5, LED1, R19, R20, U$3

Commit message: PCB updated
Parts:
- added L2: COILCRAFT-LPS4018, passives:COILCRAFT-LPS4018
- added R28: 0R, rcl:R-EU_R0603
- added R29: 0R, rcl:R-EU_R0402
Connections:
- new net N$26: L2.2, U$6.L2
- new net N$27: L2.1, U$6.L1
- net 3V: now also R29.2
- net ENUSB_CPU: now also R28.2
- net GND: now also R28.1
- net USBFAULT: now also R29.1
Other:
- moved on the sheet: C30, C31, R22, R23
Changed lines of the file:
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@@
 <part name="C39" library="rcl" deviceset="R-EU_" device="R0402"/>
 <part name="GND47" library="supply1" deviceset="GND" device=""/>
+<part name="L2" library="passives" deviceset="COILCRAFT-LPS4018" device=""/>
+<part name="R28" library="rcl" deviceset="R-EU_" device="R0603" value="0R"/>
+<part name="GND48" library="supply1" deviceset="GND" device=""/>
+<part name="R29" library="rcl" deviceset="R-EU_" device="R0402" value="0R"/>
 </parts>
 <sheets>
@@
 <instance part="C29" gate="G$1" x="311.912" y="137.16"/>
 <instance part="GND32" gate="1" x="311.912" y="127"/>
-<instance part="C30" gate="G$1" x="408.94" y="419.1"/>
-<instance part="GND33" gate="1" x="408.94" y="408.94"/>
-<instance part="C31" gate="G$1" x="401.32" y="419.1"/>
-<instance part="GND34" gate="1" x="401.32" y="408.94"/>
+<instance part="C30" gate="G$1" x="411.48" y="419.1"/>
+<instance part="GND33" gate="1" x="411.48" y="408.94"/>
+<instance part="C31" gate="G$1" x="403.86" y="419.1"/>
+<instance part="GND34" gate="1" x="403.86" y="408.94"/>
 <instance part="R21" gate="G$1" x="378.46" y="411.48" rot="R90"/>
 <instance part="GND36" gate="1" x="378.46" y="401.32"/>
@@
 <instance part="C33" gate="G$1" x="238.76" y="350.52"/>
 <instance part="GND38" gate="1" x="238.76" y="340.36"/>
-<instance part="R22" gate="G$1" x="381" y="436.88" rot="R90"/>
-<instance part="R23" gate="G$1" x="388.62" y="436.88" rot="R90"/>
+<instance part="R22" gate="G$1" x="381" y="441.96" rot="R90"/>
+<instance part="R23" gate="G$1" x="391.16" y="441.96" rot="R90"/>
 <instance part="U$6" gate="G$1" x="160.02" y="353.06"/>
 <instance part="GND39" gate="1" x="185.42" y="340.36"/>
@@
 <instance part="C39" gate="G$1" x="207.772" y="342.9"/>
 <instance part="GND47" gate="1" x="207.772" y="332.74"/>
+<instance part="L2" gate="G$1" x="160.02" y="368.3" rot="R90"/>
+<instance part="R28" gate="G$1" x="386.08" y="411.48" rot="R90"/>
+<instance part="GND48" gate="1" x="386.08" y="401.32"/>
+<instance part="R29" gate="G$1" x="398.78" y="457.2" rot="R90"/>
 </instances>
 <busses>
@@
 <pinref part="C30" gate="G$1" pin="-"/>
 <pinref part="GND33" gate="1" pin="GND"/>
-<wire x1="408.94" y1="411.48" x2="408.94" y2="414.02" width="0.1524" layer="91"/>
+<wire x1="411.48" y1="411.48" x2="411.48" y2="414.02" width="0.1524" layer="91"/>
 </segment>
 <segment>
 <pinref part="C31" gate="G$1" pin="2"/>
 <pinref part="GND34" gate="1" pin="GND"/>
-<wire x1="401.32" y1="411.48" x2="401.32" y2="414.02" width="0.1524" layer="91"/>
+<wire x1="403.86" y1="411.48" x2="403.86" y2="414.02" width="0.1524" layer="91"/>
 </segment>
 <segment>
@@
 <pinref part="GND47" gate="1" pin="GND"/>
 <wire x1="207.772" y1="335.28" x2="212.852" y2="342.9" width="0.1524" layer="91"/>
+</segment>
+<segment>
+<pinref part="R28" gate="G$1" pin="1"/>
+<pinref part="GND48" gate="1" pin="GND"/>
+<wire x1="386.08" y1="403.86" x2="386.08" y2="406.4" width="0.1524" layer="91"/>
 </segment>
 </net>
@@
 <label x="127" y="25.4" size="1.4224" layer="95" rot="R90" xref="yes"/>
 </segment>
+<segment>
+<pinref part="R29" gate="G$1" pin="2"/>
+<wire x1="398.78" y1="462.28" x2="398.78" y2="467.36" width="0.1524" layer="91"/>
+</segment>
 </net>
 <net name="_5V" class="0">
@@
 <pinref part="U$5" gate="G$1" pin="USB"/>
 <pinref part="C30" gate="G$1" pin="+"/>
-<wire x1="375.92" y1="426.72" x2="408.94" y2="426.72" width="0.1524" layer="91"/>
-<wire x1="408.94" y1="426.72" x2="408.94" y2="421.64" width="0.1524" layer="91"/>
-<wire x1="408.94" y1="426.72" x2="414.02" y2="426.72" width="0.1524" layer="91"/>
-<junction x="408.94" y="426.72"/>
+<wire x1="375.92" y1="426.72" x2="411.48" y2="426.72" width="0.1524" layer="91"/>
+<wire x1="411.48" y1="426.72" x2="411.48" y2="421.64" width="0.1524" layer="91"/>
+<wire x1="411.48" y1="426.72" x2="416.56" y2="426.72" width="0.1524" layer="91"/>
+<junction x="411.48" y="426.72"/>
 </segment>
 </net>
@@
 <net name="N$22" class="0">
 <segment>
-<wire x1="414.02" y1="429.26" x2="401.32" y2="429.26" width="0.1524" layer="91"/>
+<wire x1="416.56" y1="429.26" x2="403.86" y2="429.26" width="0.1524" layer="91"/>
 <pinref part="U$5" gate="G$1" pin="AUX"/>
 <pinref part="C31" gate="G$1" pin="1"/>
-<wire x1="401.32" y1="429.26" x2="375.92" y2="429.26" width="0.1524" layer="91"/>
-<wire x1="401.32" y1="421.64" x2="401.32" y2="429.26" width="0.1524" layer="91"/>
-<junction x="401.32" y="429.26"/>
+<wire x1="403.86" y1="429.26" x2="375.92" y2="429.26" width="0.1524" layer="91"/>
+<wire x1="403.86" y1="421.64" x2="403.86" y2="429.26" width="0.1524" layer="91"/>
+<junction x="403.86" y="429.26"/>
 </segment>
 </net>
@@
 <pinref part="U$5" gate="G$1" pin="!FAULT"/>
 <wire x1="375.92" y1="424.18" x2="381" y2="424.18" width="0.1524" layer="91"/>
-<label x="381" y="424.18" size="1.4224" layer="95" xref="yes"/>
 <pinref part="R22" gate="G$1" pin="1"/>
-<wire x1="381" y1="431.8" x2="381" y2="424.18" width="0.1524" layer="91"/>
+<wire x1="381" y1="436.88" x2="381" y2="424.18" width="0.1524" layer="91"/>
 </segment>
 </net>
@@
 <segment>
 <pinref part="U$5" gate="G$1" pin="ENUSB"/>
-<label x="381" y="421.64" size="1.4224" layer="95" xref="yes"/>
 <pinref part="R23" gate="G$1" pin="1"/>
-<wire x1="375.92" y1="421.64" x2="388.62" y2="421.64" width="0.1524" layer="91"/>
-<wire x1="388.62" y1="421.64" x2="388.62" y2="431.8" width="0.1524" layer="91"/>
+<wire x1="375.92" y1="421.64" x2="391.16" y2="421.64" width="0.1524" layer="91"/>
+<wire x1="391.16" y1="421.64" x2="391.16" y2="431.8" width="0.1524" layer="91"/>
+<pinref part="R29" gate="G$1" pin="1"/>
+<wire x1="391.16" y1="431.8" x2="391.16" y2="436.88" width="0.1524" layer="91"/>
+<wire x1="398.78" y1="452.12" x2="398.78" y2="431.8" width="0.1524" layer="91"/>
+<wire x1="398.78" y1="431.8" x2="391.16" y2="431.8" width="0.1524" layer="91"/>
+<junction x="391.16" y="431.8"/>
 </segment>
 </net>
@@
 <segment>
 <pinref part="R22" gate="G$1" pin="2"/>
-<wire x1="381" y1="441.96" x2="381" y2="444.5" width="0.1524" layer="91"/>
+<wire x1="381" y1="447.04" x2="381" y2="449.58" width="0.1524" layer="91"/>
+<label x="381" y="452.12" size="1.4224" layer="95" rot="R90" xref="yes"/>
+<pinref part="R28" gate="G$1" pin="2"/>
+<wire x1="381" y1="449.58" x2="381" y2="452.12" width="0.1524" layer="91"/>
+<wire x1="386.08" y1="416.56" x2="386.08" y2="449.58" width="0.1524" layer="91"/>
+<wire x1="386.08" y1="449.58" x2="381" y2="449.58" width="0.1524" layer="91"/>
+<junction x="381" y="449.58"/>
 </segment>
 <segment>
@@
 <segment>
 <pinref part="R23" gate="G$1" pin="2"/>
-<wire x1="388.62" y1="441.96" x2="388.62" y2="444.5" width="0.1524" layer="91"/>
+<label x="391.16" y="452.12" size="1.4224" layer="95" rot="R90" xref="yes"/>
+<wire x1="391.16" y1="447.04" x2="391.16" y2="452.12" width="0.1524" layer="91"/>
 </segment>
 <segment>
@@
 </segment>
 </net>
+<net name="N$26" class="0">
+<segment>
+<pinref part="L2" gate="G$1" pin="2"/>
+<wire x1="167.64" y1="368.3" x2="185.42" y2="368.3" width="0.1524" layer="91"/>
+<wire x1="185.42" y1="368.3" x2="185.42" y2="358.14" width="0.1524" layer="91"/>
+<pinref part="U$6" gate="G$1" pin="L2"/>
+<wire x1="185.42" y1="358.14" x2="182.88" y2="358.14" width="0.1524" layer="91"/>
+</segment>
+</net>
+<net name="N$27" class="0">
+<segment>
+<pinref part="L2" gate="G$1" pin="1"/>
+<wire x1="152.4" y1="368.3" x2="134.62" y2="368.3" width="0.1524" layer="91"/>
+<wire x1="134.62" y1="368.3" x2="134.62" y2="358.14" width="0.1524" layer="91"/>
+<pinref part="U$6" gate="G$1" pin="L1"/>
+<wire x1="134.62" y1="358.14" x2="137.16" y2="358.14" width="0.1524" layer="91"/>
+</segment>
+</net>

Commit message: PCB Updated
Parts:
- added PAD1, PAD2: WIREPADSMD1,27-254, wirepad:WIREPADSMD1,27-254
- added R30, R31, R32: (no value), rcl:R-EU_R0603
- added R33: (no value), rcl:R-EU_M0805
- C39: device rcl:R-EU_R0402 -> rcl:C-EUC0402
- R29: device rcl:R-EU_R0402 -> rcl:R-EU_R0603
Connections:
- removed net POWER_EN: U$2.PC6, U$6.EN
- new net ADC1_IN2: R31.2, R32.1, U$2.PA2
- new net CHARGING: R30.1, U$2.PA9
- new net N$28: R33.2, U$2.VDDA
- net 3V: now also R33.1
- net GND: now also PAD2.P, R32.2
- net LCD_BACKLIGHT: now also U$2.PC6; no longer U$2.PB10
- net LIPOL: now also PAD1.P, R31.1, U$6.EN
- net N$18: now also R30.2
Other:
- moved on the sheet: C27, C28, C39, F3, JP5, LED1, R19, R20, U$3

Commit message: PCB Updated
Parts:
- added C40, C41: (no value), rcl:C-EUC0402
- added C42: (no value), rcl:C-EUC0603
- added R34: 0R, rcl:R-EU_R0603
- added S1: SWS001, smd-special:SWS001
Connections:
- new net N$29: R34.1, S1.1, U$2.BOOT0
- net 3V: now also C41.1, S1.2
- net ADC1_IN2: now also C42.1
- net GND: now also C40.2, C41.2, C42.2, R34.2, U$2.PDR_ON
- net N$28: now also C40.1, U$2.VREF+
Other:
- moved on the sheet: C15, C16, C17, C18, C3, C4, L1

Commit message: Rotary encoder added
Parts:
- removed C1, C2: 22 pF, rcl:C-EUC0603
- removed Y1: CRYSTAL-GROUNDEDSMD-5X3.2, SparkFun-Clocks:CRYSTAL-GROUNDEDSMD-5X3.2
- added C43: (no value), rcl:CPOL-EUSMCA
- added R35: (no value), rcl:R-EU_R0603
- added U$7: ASE, crystal:ASE
- U$4: value EVQWK -> EVQWKSMD; device mw:EVQWK -> mw:EVQWKSMD
Connections:
- new net SW2: U$2.PB9, U$4.SW2
- new net SW_A: U$2.PE2, U$4.A
- new net SW_B: U$2.PB8, U$4.B
- net 3V: now also C43.+, R35.2, U$7.VDD
- net GND: now also C43.-, U$4.MNT, U$7.GND; no longer C1.2, C2.2, Y1.3
- net NRST: now also R35.1
- net PH0: now also U$7.OUT; no longer C2.1, Y1.2
- net PH1: no longer C1.1, Y1.1
Other:
- moved on the sheet: C15, C16, C17, C18, C19, C20, C21, C22, C41, JP1, L1
