File: hardware/whypod.brd (EAGLE design)
At the start: 68.2 x 104.8 mm, 70 parts, among them IC1 IC_USBLC6-2, J1 AUDIO_JACK_TRRSSMD_RA, U1 USD-SOCKETUSD, X2 USB-A-S, Y1 CRYSTAL-GROUNDEDSMD-5X3.2, Y2 CRYSTAL-GROUNDEDSMD-5X3.2

Commit message: USB power supply
Parts:
- added C31: (no value), rcl:C0603
- added R21: (no value), rcl:R0603
- C30: device rcl:SMC_E -> rcl:SMC_D
- moved U$5 2.50 mm to (49.5, 37.2)
- moved C30 2.46 mm to (53.2, 43.2), turned to 0 degrees
Connections:
- new net N$21: R21.2, U$5.6
- net GND: now also C31.2, R21.1
- net N$22: now also C31.1
Routing:
- net _5V: track 7.96 -> 20.3 mm
- net USBFAULT: track 21.8 -> 29.3 mm
- net ENUSB: track 19.4 -> 25.5 mm
- net N$21: track 0.00 -> 1.65 mm
- net N$22: track 0.00 -> 1.53 mm
- net GND: track 33.8 -> 34.1 mm, vias 16 -> 18
Changed lines of the file:
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@@
 <text x="40.64" y="60.96" size="1.778" layer="1">SQ9RZI</text>
 <rectangle x1="-1.905" y1="19.685" x2="2.54" y2="29.845" layer="41"/>
-<rectangle x1="49.1998" y1="37.7698" x2="52.3748" y2="40.9448" layer="41" rot="R90"/>
+<rectangle x1="47.9298" y1="35.6108" x2="51.1048" y2="38.7858" layer="41" rot="R90"/>
 </plain>
 <attributes>
@@
 </element>
 <element name="U$4" library="mw" package="EVQWK" value="EVQWK" x="3.365" y="64.135"/>
-<element name="U$5" library="mw" package="DRC10" value="TPS2500" x="50.8" y="39.37" rot="R90"/>
+<element name="U$5" library="mw" package="DRC10" value="TPS2500" x="49.53" y="37.211" rot="R90"/>
 <element name="C29" library="rcl" package="C0603" value="" x="49.1932" y="50.8896" rot="R180"/>
-<element name="C30" library="rcl" package="SMC_E" value="" x="50.8" y="43.815" rot="R180"/>
+<element name="C30" library="rcl" package="SMC_D" value="" x="53.1876" y="43.2308"/>
+<element name="C31" library="rcl" package="C0603" value="" x="51.7779" y="39.878"/>
+<element name="R21" library="rcl" package="R0603" value="" x="46.4312" y="39.0144"/>
 </elements>
 <signals>
@@
 <contactref element="U$5" pad="5"/>
 <contactref element="U$5" pad="T"/>
-<wire x1="49.8" y1="38.07" x2="49.8" y2="36.9156" width="0.3048" layer="1"/>
-<wire x1="49.8" y1="36.9156" x2="49.8348" y2="36.8808" width="0.3048" layer="1"/>
-<wire x1="50.8" y1="39.37" x2="48.26" y2="39.37" width="1.016" layer="1"/>
-<wire x1="50.8" y1="39.37" x2="53.34" y2="39.37" width="1.016" layer="1"/>
+<wire x1="49.53" y1="37.211" x2="48.7934" y2="37.211" width="1.016" layer="1"/>
+<wire x1="48.7934" y1="37.211" x2="46.9646" y2="37.1856" width="1.016" layer="1"/>
+<wire x1="49.53" y1="37.211" x2="50.0634" y2="37.211" width="1.016" layer="1"/>
 <contactref element="U$5" pad="2"/>
-<wire x1="51.3" y1="38.07" x2="51.3" y2="36.9744" width="0.3048" layer="1"/>
-<wire x1="51.3" y1="36.9744" x2="51.2064" y2="36.8808" width="0.3048" layer="1"/>
+<wire x1="50.0634" y1="37.211" x2="52.1208" y2="37.211" width="1.016" layer="1"/>
 <contactref element="C29" pad="2"/>
 <contactref element="C30" pad="-"/>
+<contactref element="C31" pad="2"/>
+<via x="47.8282" y="47.6504" extent="1-16" drill="0.6" diameter="1.4224" shape="octagon"/>
+<wire x1="48.53" y1="35.911" x2="48.53" y2="36.9476" width="0.3048" layer="1"/>
+<wire x1="48.53" y1="36.9476" x2="48.7934" y2="37.211" width="0.3048" layer="1"/>
+<wire x1="50.03" y1="35.911" x2="50.03" y2="37.1776" width="0.3048" layer="1"/>
+<wire x1="50.03" y1="37.1776" x2="50.0634" y2="37.211" width="0.3048" layer="1"/>
+<contactref element="R21" pad="1"/>
+<via x="52.1208" y="37.211" extent="1-16" drill="0.6" diameter="1.4224" shape="octagon"/>
 </signal>
 <signal name="DB0">
@@
 <wire x1="48.895" y1="53.79211875" x2="49.6062" y2="53.79211875" width="0.4064" layer="1"/>
 <wire x1="50.045" y1="53.35331875" x2="49.6062" y2="53.79211875" width="0.4064" layer="1"/>
-<wire x1="53.95" y1="43.815" x2="54.1064" y2="50.8896" width="0" layer="19" extent="1-1"/>
-<wire x1="51.3" y1="40.67" x2="53.95" y2="43.815" width="0" layer="19" extent="1-1"/>
+<wire x1="50.0432" y1="50.8896" x2="50.0432" y2="43.2364" width="0.6096" layer="1"/>
+<wire x1="50.0432" y1="43.2364" x2="50.0376" y2="43.2308" width="0.6096" layer="1"/>
+<wire x1="50.03" y1="38.511" x2="50.03" y2="43.2232" width="0.3048" layer="1"/>
+<wire x1="50.03" y1="43.2232" x2="50.0376" y2="43.2308" width="0.3048" layer="1"/>
 </signal>
 <signal name="N$1">
@@
 <signal name="N$22">
 <contactref element="U$5" pad="10"/>
+<contactref element="C31" pad="1"/>
+<wire x1="50.53" y1="38.511" x2="50.53" y2="39.4801" width="0.3048" layer="1"/>
+<wire x1="50.53" y1="39.4801" x2="50.9279" y2="39.878" width="0.3048" layer="1"/>
 </signal>
 <signal name="N$23">
 <contactref element="U$5" pad="4"/>
 <contactref element="U$5" pad="3"/>
-<wire x1="50.3" y1="38.07" x2="50.8" y2="38.07" width="0" layer="19" extent="1-1"/>
+<wire x1="49.53" y1="35.911" x2="49.03" y2="35.911" width="0" layer="19" extent="1-1"/>
 </signal>
 <signal name="ENUSB">
@@
 <wire x1="32.3118" y1="50.6396" x2="41.0798" y2="50.6396" width="0.3048" layer="1"/>
 <wire x1="41.0798" y1="50.6396" x2="45.1358" y2="46.5836" width="0.3048" layer="1"/>
-<wire x1="45.1358" y1="46.5836" x2="45.1358" y2="42.4942" width="0.3048" layer="1"/>
-<wire x1="45.1358" y1="42.4942" x2="45.72" y2="41.91" width="0.3048" layer="1"/>
-<wire x1="45.72" y1="41.91" x2="50.3" y2="40.67" width="0" layer="19" extent="1-1"/>
+<wire x1="45.1358" y1="46.5836" x2="45.1358" y2="41.2242" width="0.3048" layer="1"/>
+<wire x1="49.03" y1="38.511" x2="49.03" y2="39.6414" width="0.3048" layer="1"/>
+<wire x1="49.03" y1="39.6414" x2="48.641" y2="40.0304" width="0.3048" layer="1"/>
+<wire x1="48.641" y1="40.0304" x2="46.3296" y2="40.0304" width="0.3048" layer="1"/>
+<wire x1="46.3296" y1="40.0304" x2="45.1358" y2="41.2242" width="0.3048" layer="1"/>
 </signal>
 <signal name="USBFAULT">
@@
 <wire x1="32.3118" y1="52.1396" x2="44.6344" y2="52.1396" width="0.3048" layer="1"/>
 <wire x1="44.6344" y1="52.1396" x2="45.7454" y2="51.0286" width="0.3048" layer="1"/>
-<wire x1="45.7454" y1="51.0286" x2="45.7454" y2="43.1546" width="0.3048" layer="1"/>
-<wire x1="45.7454" y1="43.1546" x2="50.8" y2="40.67" width="0" layer="19" extent="1-1"/>
+<wire x1="45.7454" y1="51.0286" x2="45.7454" y2="41.4782" width="0.3048" layer="1"/>
+<wire x1="49.53" y1="38.511" x2="49.53" y2="40.005" width="0.3048" layer="1"/>
+<wire x1="49.53" y1="40.005" x2="48.895" y2="40.64" width="0.3048" layer="1"/>
+<wire x1="48.895" y1="40.64" x2="46.5836" y2="40.64" width="0.3048" layer="1"/>
+<wire x1="46.5836" y1="40.64" x2="45.7454" y2="41.4782" width="0.3048" layer="1"/>
+</signal>
+<signal name="N$21">
+<contactref element="U$5" pad="6"/>
+<contactref element="R21" pad="2"/>
+<wire x1="48.53" y1="38.511" x2="48.53" y2="38.846" width="0.3048" layer="1"/>
+<wire x1="48.53" y1="38.846" x2="48.3616" y2="39.0144" width="0.3048" layer="1"/>
+<wire x1="48.3616" y1="39.0144" x2="47.2812" y2="39.0144" width="0.3048" layer="1"/>
 </signal>
 </signals>

Commit message: Power circuit updated
Parts:
- added C32: (no value), rcl:C0603
- added C33: (no value), rcl:SMC_C
- added L3: COILCRAFT-LPS4018, passives:LPS4018
- added R22, R23: 0R, rcl:R0603
- moved JP5 68.3 mm to (65.4, 39.4), turned to 180 degrees
- moved LED1 63.9 mm to (65.6, 32.8), turned to 180 degrees
- moved R20 58.6 mm to (63.3, 32.1), turned to 180 degrees
- moved F3 56.7 mm to (59.4, 38.1), turned to 0 degrees
- moved C28 55.4 mm to (56.3, 35.9), turned to 270 degrees
- moved R19 54.0 mm to (58.5, 40.0), turned to 0 degrees
- moved C27 52.0 mm to (53.0, 36.4)
- moved U$3 50.8 mm to (55.1, 39.0), turned to 270 degrees
- moved C31 6.13 mm to (45.8, 41.2), turned to 180 degrees
- moved R21 5.97 mm to (52.0, 41.2), turned to 180 degrees
- moved U$5 2.30 mm to (48.9, 39.4)
- moved C30 2.08 mm to (51.5, 44.5)
Connections:
- removed net N$23: U$5.3, U$5.4
- removed net VBAT: C27.1, U$3.3
- new net ENUSB_CPU: R22.2, U$2.PC7
- new net LIPOL: C27.1, C32.1, L3.1, U$3.3, U$5.3, U$5.4
- new net N$24: L3.2, U$5.1
- new net USBFAULT_CPU: R23.2, U$2.PA8
- net 3V: now also C33.+
- net ENUSB: now also R22.1, U$5.8; no longer U$2.PC7, U$5.7
- net GND: now also C32.2, C33.-
- net USBFAULT: now also R23.1, U$5.7; no longer U$2.PA8, U$5.8
Routing:
- net USBFAULT_CPU: track 0.00 -> 18.8 mm
- net USBFAULT: track 29.3 -> 10.8 mm
- net ENUSB_CPU: track 0.00 -> 18.1 mm
- net ENUSB: track 25.5 -> 7.76 mm
- net NRST: track 0.00 -> 16.4 mm
- net LIPOL: track 0.00 -> 13.8 mm
- net N$18: track 1.52 -> 14.9 mm
- net VBUS: track 3.84 -> 14.3 mm
- net N$24: track 0.00 -> 5.40 mm
- net 3V: track 219.6 -> 221.9 mm
- net VBAT: track 1.78 -> 0.00 mm
- net _5V: track 20.3 -> 18.8 mm
- net N$19: track 0.00 -> 1.44 mm
- net GND: track 34.1 -> 34.2 mm, vias 18 -> 20

Commit message: PCB updated
Parts:
- added C34, C35, C36, C37: (no value), rcl:C0805
- added C38: (no value), rcl:C0603
- added C39, R24, R27: (no value), rcl:R0402
- added U$6: TPS63060, mw:DRC10
- C33: device rcl:SMC_C -> rcl:C0805
- R12: device rcl:R0603 -> rcl:R0402
- moved C33 5.22 mm to (58.5, 24.2), turned to 90 degrees
- moved C4 0.71 mm to (35.7, 56.4)
- moved R12 0.55 mm to (54.6, 19.5)
Connections:
- new net N$23: C38.1, U$6.6
- new net N$25: C39.1, R24.2, R27.1, U$6.8
- new net POWER_EN: U$2.PC6, U$6.3
- net 3V: now also C33.1, C34.1, C35.1, R27.2, U$6.9; no longer C33.+
- net GND: now also C33.2, C34.2, C35.2, C36.2, C37.2, C38.2, C39.2, R24.1, U$6.4, U$6.7, U$6.T; no longer C33.-
- net LCD_BACKLIGHT: now also U$2.PB10; no longer U$2.PC6
- net LIPOL: now also C36.1, C37.1, U$6.2
Routing:
- net POWER_EN: track 0.00 -> 41.0 mm
- net 3V: track 221.9 -> 230.0 mm
- net LIPOL: track 13.8 -> 21.3 mm
- net N$25: track 0.00 -> 4.14 mm
- net GND: track 34.2 -> 38.1 mm, vias 20 -> 21
- net LCD_BACKLIGHT: track 45.5 -> 42.9 mm, vias 0 -> 2
- net N$23: track 0.00 -> 1.27 mm
- net N$7: track 4.28 -> 3.57 mm
- net N$11: track 13.9 -> 13.4 mm

Commit message: PCB updated
Parts:
- added L2: COILCRAFT-LPS4018, passives:LPS4018
- added R28: 0R, rcl:R0603
- added R29: 0R, rcl:R0402
- moved C35 6.59 mm to (59.0, 18.7), turned to 0 degrees
- moved C34 3.83 mm to (59.0, 20.7), turned to 0 degrees
- moved C36 2.56 mm to (57.3, 29.3)
- moved C37 2.56 mm to (57.3, 31.2)
- moved C38 2.54 mm to (52.3, 24.7)
- moved C39 2.54 mm to (54.5, 23.4)
- moved R24 2.54 mm to (54.5, 22.1)
- moved R27 2.54 mm to (56.4, 22.7)
- moved U$6 2.54 mm to (55.4, 26.0)
- moved C33 1.54 mm to (59.0, 22.8), turned to 0 degrees
Connections:
- new net N$26: L2.2, U$6.10
- new net N$27: L2.1, U$6.1
- net 3V: now also R29.2
- net ENUSB_CPU: now also R28.2
- net GND: now also R28.1
- net USBFAULT: now also R29.1
Routing:
- net N$27: track 0.00 -> 3.04 mm
- net N$26: track 0.00 -> 3.04 mm
- net POWER_EN: track 41.0 -> 43.7 mm
- net 3V: track 230.0 -> 232.3 mm, vias 6 -> 7
- net LIPOL: track 21.3 -> 23.3 mm
- net USBFAULT: track 10.8 -> 12.7 mm, vias 0 -> 1
- net GND: vias 21 -> 23

Commit message: PCB Updated
Parts:
- added PAD1, PAD2: WIREPADSMD1,27-254, wirepad:SMD1,27-2,54
- added R30, R31, R32: (no value), rcl:R0603
- added R33: (no value), rcl:M0805
- C39: device rcl:R0402 -> rcl:C0402
- R29: device rcl:R0402 -> rcl:R0603
- moved C29 3.17 mm to (49.2, 54.1)
- moved IC1 3.17 mm to (48.9, 57.1)
- moved X2 3.17 mm to (57.6, 57.1)
- moved R29 3.12 mm to (52.4, 46.9), turned to 270 degrees
- moved R20 2.67 mm to (64.8, 29.9), turned to 270 degrees
- moved JP1 1.91 mm to (59.5, 80.0)
- moved T1 1.56 mm to (55.3, 7.06), flipped to the top, turned to 90 degrees
- moved C38 1.42 mm to (52.9, 26.0)
- moved U$6 1.42 mm to (56.0, 27.3)
- moved C33 1.42 mm to (59.6, 24.0)
- moved C34 1.42 mm to (59.6, 22.0)
- moved C35 1.42 mm to (59.6, 20.0)
- moved C36 1.42 mm to (58.0, 30.6)
- moved C37 1.42 mm to (58.0, 32.5)
- moved C39 1.42 mm to (55.2, 24.7)
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Connections:
- removed net POWER_EN: U$2.PC6, U$6.3
- new net ADC1_IN2: R31.2, R32.1, U$2.PA2
- new net CHARGING: R30.1, U$2.PA9
- new net N$28: R33.2, U$2.VDDA
- net 3V: now also R33.1
- net GND: now also PAD2.1, R32.2
- net LCD_BACKLIGHT: now also U$2.PC6; no longer U$2.PB10
- net LIPOL: now also PAD1.1, R31.1, U$6.3
- net N$18: now also R30.2
Routing:
- net 3V: track 232.3 -> 304.6 mm, vias 7 -> 8
- net ADC1_IN2: track 0.00 -> 49.8 mm, vias 0 -> 1
- net POWER_EN: track 43.7 -> 0.00 mm
- net N$18: track 14.9 -> 36.3 mm
- net CHARGING: track 0.00 -> 17.6 mm
- net N$28: track 0.00 -> 11.5 mm
- net _5V: track 18.8 -> 22.0 mm
- net LCD_BACKLIGHT: track 43.1 -> 45.9 mm, vias 2 -> 0
- net GND: track 38.1 -> 40.1 mm, vias 23 -> 24
- net LIPOL: track 23.3 -> 24.8 mm
- net LED_A: track 5.92 -> 4.44 mm, vias 1 -> 0
- net USB_D_P: track 16.9 -> 18.2 mm
- net USB_D_N: track 16.9 -> 18.2 mm
- net N$11: track 13.4 -> 14.4 mm, vias 1 -> 0
- net SWD_IO: track 34.9 -> 35.7 mm
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
Commit message: PCB Updated
Parts:
- added C40, C41: (no value), rcl:C0402
- added C42: (no value), rcl:C0603
- added R34: 0R, rcl:R0603
- added S1: SWS001, smd-special:SMS-001
- moved C22 4.72 mm to (17.0, 69.6), turned to 270 degrees
- moved R32 1.93 mm to (48.0, 28.1), turned to 0 degrees
- moved C7 1.91 mm to (12.1, 52.4)
- moved Y1 1.91 mm to (8.64, 50.4)
- moved C1 1.90 mm to (3.81, 49.3)
- moved C2 1.90 mm to (3.81, 51.5)
- moved R31 0.99 mm to (48.0, 30.0), turned to 180 degrees
Connections:
- new net N$29: R34.1, S1.1, U$2.BOOT0
- net 3V: now also C41.1, S1.2
- net ADC1_IN2: now also C42.1
- net GND: now also C40.2, C41.2, C42.2, R34.2, U$2.PDR_ON
- net N$28: now also C40.1, U$2.VREF+
Routing:
- net 3V: track 304.6 -> 374.9 mm, vias 8 -> 9
- net N$29: track 0.00 -> 45.3 mm
- net ADC1_IN2: track 49.8 -> 64.3 mm, vias 1 -> 2
- net GND: track 40.1 -> 44.9 mm, vias 24 -> 25
- net LIPOL: track 24.8 -> 27.3 mm
- net NRST: track 16.4 -> 18.3 mm
- net PH1: track 12.2 -> 14.1 mm
- net PH0: track 12.2 -> 14.1 mm
- net N$28: track 11.5 -> 13.0 mm

Commit message: PCB updated
Parts:
- moved R6 5.70 mm to (53.2, 87.8), flipped to the top, turned to 0 degrees
- moved R3 2.32 mm to (52.4, 85.9), flipped to the top, turned to 0 degrees
Routing:
- net NRST: track 18.3 -> 71.8 mm, vias 0 -> 1
- net SDIO_D1: track 82.2 -> 77.3 mm
- net SDIO_D0: track 82.5 -> 78.0 mm
- net LCD_CS: track 87.7 -> 86.7 mm
- net SWD_IO: track 35.7 -> 34.7 mm
- net LCD_WR: track 73.7 -> 73.0 mm
- net LCD_RD: track 66.1 -> 65.5 mm
- net I2S_WS: track 36.4 -> 36.9 mm, vias 5 -> 2
- net GND: vias 25 -> 24

Commit message: Rotary encoder added
Parts:
- removed C1, C2: 22 pF, rcl:C0603
- removed Y1: CRYSTAL-GROUNDEDSMD-5X3.2, SparkFun-Clocks:CRYSTAL-SMD-5X3.2-4PAD
- added C43: (no value), rcl:SMC_A
- added R35: (no value), rcl:R0603
- added U$7: ASE, crystal:ASE
- U$4: value EVQWK -> EVQWKSMD; device mw:EVQWK -> mw:EVQWK_SMD
- moved C8 2.20 mm to (16.0, 57.9)
- moved C7 1.91 mm to (14.0, 52.4)
- moved U$4 0.23 mm to (3.37, 63.9)
Connections:
- new net SW2: U$2.PB9, U$4.SW2
- new net SW_A: U$2.PE2, U$4.A
- new net SW_B: U$2.PB8, U$4.B
- net 3V: now also C43.+, R35.2, U$7.4
- net GND: now also C43.-, U$4.NC1, U$4.NC2, U$7.2; no longer C1.2, C2.2, Y1.2, Y1.4
- net NRST: now also R35.1
- net PH0: now also U$7.3; no longer C2.1, Y1.1
- net PH1: no longer C1.1, Y1.3
Routing:
- net SW_B: track 0.00 -> 15.2 mm
- net PH1: track 14.1 -> 0.00 mm
- net SW2: track 0.00 -> 12.2 mm
- net PH0: track 14.1 -> 6.36 mm
- net NRST: track 71.8 -> 65.2 mm, vias 1 -> 2
- net 3V: track 375.1 -> 381.3 mm
- net SW_A: track 0.00 -> 5.32 mm
- net GND: track 44.9 -> 42.1 mm, vias 24 -> 26
- net N$29: track 45.3 -> 44.5 mm
