File: hardware/whypod.brd (EAGLE design)
At the start: 68.2 x 104.8 mm, 118 parts, among them IC1 IC_USBLC6-2, J1 AUDIO_JACK_TRRSSMD_RA, U1 USD-SOCKETUSD, X1 CRYSTALS-NOGND-CFPX-217, X2 USB-A-S, Y2 CRYSTAL-GROUNDEDSMD-5X3.2

Commit message: Some minor changes
Parts:
- removed R34: 0R, rcl:R0603
- removed S1: SWS001, smd-special:SMS-001
Connections:
- removed net N$29: R34.1, S1.1, U$2.BOOT0
- net 3V: no longer S1.2
- net GND: now also U$2.BOOT0; no longer R34.2
Routing:
- net N$29: track 44.5 -> 0.00 mm
- net 3V: track 397.2 -> 382.9 mm
- net GND: track 47.4 -> 55.5 mm, vias 29 -> 28
Changed lines of the file:
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@@
 <circle x="3.89" y="16.51" radius="1.778" width="0.254" layer="42"/>
 <circle x="64.69" y="16.51" radius="1.778" width="0.254" layer="42"/>
+<rectangle x1="22.86" y1="57.288734375" x2="24.13" y2="57.785" layer="41"/>
 </plain>
 <attributes>
@@
 <element name="C41" library="rcl" package="C0402" value="" x="13.335" y="46.2915" rot="R270"/>
 <element name="C42" library="rcl" package="C0603" value="" x="49.95" y="26.1112"/>
-<element name="R34" library="rcl" package="R0603" value="0R" x="6.5532" y="87.9165125" rot="R90"/>
-<element name="S1" library="smd-special" package="SMS-001" value="SWS001" x="6.5532" y="80.5688" rot="R180"/>
 <element name="C43" library="rcl" package="SMC_A" value="" x="61.8236" y="87.8332"/>
 <element name="U$7" library="crystal" package="ASE" value="ASE" x="9.4742" y="48.7">
@@
 <contactref element="U$2" pad="PDR_ON"/>
 <contactref element="C42" pad="2"/>
-<contactref element="R34" pad="2"/>
-<via x="20.1558" y="66.4972" extent="1-16" drill="0.6" diameter="1.4224" shape="octagon"/>
+<via x="18.8858" y="66.2178" extent="1-16" drill="0.6" diameter="1.4224" shape="octagon"/>
 <contactref element="C43" pad="-"/>
 <via x="62.4332" y="90.805" extent="1-16" drill="0.6" diameter="1.4224" shape="octagon"/>
@@
 <contactref element="U$10" pad="MNT1"/>
 <contactref element="U$10" pad="B"/>
-<via x="15.7108" y="70.3072" extent="1-16" drill="0.6" diameter="1.4224" shape="octagon"/>
 <contactref element="U$8" pad="MNT1"/>
 <contactref element="U$8" pad="MNT2"/>
@@
 <contactref element="X2" pad="P$6"/>
 <contactref element="X2" pad="P$5"/>
+<contactref element="U$2" pad="BOOT0"/>
+<wire x1="23.4668" y1="57.8896" x2="23.4668" y2="63.1218" width="0.3048" layer="1"/>
+<wire x1="23.4668" y1="63.1218" x2="21.463" y2="65.1256" width="0.3048" layer="1"/>
 </signal>
 <signal name="DB0">
@@
 <wire x1="12.7" y1="7.366" x2="12.7" y2="27.305" width="0.8128" layer="16"/>
 <via x="12.7" y="27.305" extent="1-16" drill="0.6" diameter="1.4224" shape="octagon"/>
-<wire x1="21.4828" y1="43.4594" x2="21.4828" y2="45.4434" width="0.3048" layer="1"/>
-<wire x1="21.4828" y1="45.4434" x2="19.7866" y2="47.1396" width="0.3048" layer="1"/>
+<wire x1="21.4828" y1="43.4594" x2="21.4828" y2="46.4622" width="0.3048" layer="1"/>
 <contactref element="R33" pad="1"/>
 <wire x1="20.68706875" y1="36.2712" x2="20.76326875" y2="36.195" width="0.3048" layer="1"/>
 <wire x1="20.76326875" y1="36.195" x2="21.083640625" y2="36.195" width="0.3048" layer="1"/>
 <contactref element="C41" pad="1"/>
-<contactref element="S1" pad="2"/>
 <wire x1="18.8858" y1="71.0706" x2="18.8858" y2="72.898" width="0.6096" layer="1"/>
-<wire x1="18.8858" y1="72.898" x2="7.747" y2="72.898" width="0.4064" layer="1"/>
-<wire x1="7.747" y1="72.898" x2="6.5532" y2="74.0918" width="0.4064" layer="1"/>
-<wire x1="6.5532" y1="76.073" x2="6.5532" y2="74.0918" width="0.4064" layer="1"/>
 <via x="64.6176" y="46.013" extent="1-16" drill="0.6" diameter="1.4224" shape="octagon"/>
 <wire x1="66.2432" y1="44.3874" x2="64.6176" y2="46.013" width="0.8128" layer="16"/>
@@
 <wire x1="19.9018" y1="28.1822" x2="19.0246" y2="27.305" width="0.6096" layer="1"/>
 <wire x1="19.0246" y1="27.305" x2="12.7" y2="27.305" width="0.6096" layer="1"/>
+<wire x1="19.7866" y1="47.1396" x2="20.8054" y2="47.1396" width="0.3048" layer="1"/>
+<wire x1="21.4828" y1="46.4622" x2="20.8054" y2="47.1396" width="0.3048" layer="1"/>
 </signal>
 <signal name="_5V">
@@
 <contactref element="U$2" pad="VDDA"/>
 <contactref element="R33" pad="2"/>
-<wire x1="18.7168" y1="45.6396" x2="19.685" y2="45.6396" width="0.3048" layer="1"/>
-<wire x1="19.685" y1="45.6396" x2="19.74" y2="45.6396" width="0.3048" layer="1"/>
-<wire x1="19.74" y1="45.6396" x2="20.1422" y2="45.2374" width="0.3048" layer="1"/>
-<wire x1="20.1422" y1="45.2374" x2="20.1422" y2="43.815" width="0.3048" layer="1"/>
-<wire x1="20.1422" y1="43.815" x2="18.288" y2="41.9608" width="0.3048" layer="1"/>
+<wire x1="18.7168" y1="45.6396" x2="19.7866" y2="45.6396" width="0.3048" layer="1"/>
+<wire x1="19.7866" y1="43.4594" x2="18.288" y2="41.9608" width="0.3048" layer="1"/>
 <wire x1="18.288" y1="41.9608" x2="18.288" y2="40.005" width="0.3048" layer="1"/>
 <wire x1="18.288" y1="40.005" x2="18.288" y2="36.8554" width="0.3048" layer="1"/>
@@
 <contactref element="C40" pad="1"/>
 <contactref element="U$2" pad="VREF+"/>
-<wire x1="18.7168" y1="46.1396" x2="19.685" y2="46.1396" width="0.3048" layer="1"/>
-<wire x1="19.685" y1="46.1396" x2="19.685" y2="45.6396" width="0.3048" layer="1"/>
+<wire x1="18.7168" y1="46.1396" x2="19.7866" y2="46.1396" width="0.3048" layer="1"/>
+<wire x1="19.7866" y1="46.1396" x2="19.7866" y2="45.6396" width="0.3048" layer="1"/>
 <wire x1="18.7168" y1="45.6396" x2="16.0062" y2="45.6396" width="0.3048" layer="1"/>
 <contactref element="C47" pad="1"/>
 <wire x1="17.868" y1="40.1574" x2="18.1356" y2="40.1574" width="0.3048" layer="1"/>
 <wire x1="18.1356" y1="40.1574" x2="18.288" y2="40.005" width="0.3048" layer="1"/>
+<wire x1="19.7866" y1="45.6396" x2="19.7866" y2="43.4594" width="0.3048" layer="1"/>
 </signal>
 <signal name="ADC1_IN2">
@@
 <wire x1="47.5742" y1="28.067" x2="36.2458" y2="28.067" width="0.3048" layer="16"/>
 </signal>
-<signal name="N$29">
-<contactref element="U$2" pad="BOOT0"/>
-<contactref element="R34" pad="1"/>
-<wire x1="23.4668" y1="57.8896" x2="23.4668" y2="63.1218" width="0.3048" layer="1"/>
-<contactref element="S1" pad="1"/>
-<wire x1="21.463" y1="65.1256" x2="18.161" y2="65.1256" width="0.3048" layer="1"/>
-<wire x1="23.4668" y1="63.1218" x2="21.463" y2="65.1256" width="0.3048" layer="1"/>
-<wire x1="17.3482" y1="71.4502" x2="16.6624" y2="72.136" width="0.3048" layer="1"/>
-<wire x1="16.6624" y1="72.136" x2="7.239" y2="72.136" width="0.3048" layer="1"/>
-<wire x1="7.239" y1="72.136" x2="5.5372" y2="73.8378" width="0.3048" layer="1"/>
-<wire x1="5.5372" y1="73.8378" x2="5.5372" y2="82.3214" width="0.3048" layer="1"/>
-<wire x1="6.5532" y1="85.0646" x2="6.5532" y2="83.3374" width="0.3048" layer="1"/>
-<wire x1="6.5532" y1="83.3374" x2="5.5372" y2="82.3214" width="0.3048" layer="1"/>
-<wire x1="6.5532" y1="85.0646" x2="6.5532" y2="87.0665125" width="0.6096" layer="1"/>
-<wire x1="17.3482" y1="71.4502" x2="17.3482" y2="65.9384" width="0.3048" layer="1"/>
-<wire x1="17.3482" y1="65.9384" x2="18.161" y2="65.1256" width="0.3048" layer="1"/>
-</signal>
 <signal name="SW2">
 <contactref element="U$4" pad="SW2"/>
@@
 <wire x1="13.081" y1="63.119" x2="20.8788" y2="63.119" width="0.3048" layer="1"/>
 <wire x1="13.081" y1="63.119" x2="12.065" y2="64.135" width="0.3048" layer="1"/>
-<wire x1="12.065" y1="64.135" x2="12.065" y2="69.9262" width="0.3048" layer="1"/>
-<wire x1="12.065" y1="69.9262" x2="10.4902" y2="71.501" width="0.3048" layer="1"/>
-<wire x1="10.4902" y1="71.501" x2="7.0104" y2="71.501" width="0.3048" layer="1"/>
-<wire x1="4.9276" y1="73.5838" x2="4.9276" y2="91.5924" width="0.3048" layer="1"/>
+<wire x1="12.065" y1="64.135" x2="12.065" y2="71.1962" width="0.3048" layer="1"/>
+<wire x1="12.065" y1="71.1962" x2="10.4902" y2="72.771" width="0.3048" layer="1"/>
+<wire x1="10.4902" y1="72.771" x2="6.3754" y2="72.771" width="0.3048" layer="1"/>
+<wire x1="4.9276" y1="74.2188" x2="4.9276" y2="91.5924" width="0.3048" layer="1"/>
 <wire x1="4.9276" y1="91.5924" x2="3.37" y2="93.15" width="0.3048" layer="1"/>
 <wire x1="2.3462" y1="93.15" x2="3.37" y2="93.15" width="0.3048" layer="1"/>
-<wire x1="7.0104" y1="71.501" x2="4.9276" y2="73.5838" width="0.3048" layer="1"/>
+<wire x1="6.3754" y1="72.771" x2="4.9276" y2="74.2188" width="0.3048" layer="1"/>
 </signal>
 <signal name="VOL_DN">
 <contactref element="U$10" pad="A"/>
-<wire x1="11.4554" y1="61.0362" x2="11.4554" y2="69.6722" width="0.3048" layer="1"/>
-<wire x1="11.4554" y1="69.6722" x2="10.2362" y2="70.8914" width="0.3048" layer="1"/>
-<wire x1="10.2362" y1="70.8914" x2="6.7564" y2="70.8914" width="0.3048" layer="1"/>
-<wire x1="6.7564" y1="70.8914" x2="4.318" y2="73.3298" width="0.3048" layer="1"/>
-<wire x1="4.318" y1="73.3298" x2="4.318" y2="80.899" width="0.3048" layer="1"/>
+<wire x1="11.4554" y1="61.0362" x2="11.4554" y2="70.9422" width="0.3048" layer="1"/>
+<wire x1="11.4554" y1="70.9422" x2="10.2362" y2="72.1614" width="0.3048" layer="1"/>
+<wire x1="10.2362" y1="72.1614" x2="6.1214" y2="72.1614" width="0.3048" layer="1"/>
+<wire x1="6.1214" y1="72.1614" x2="4.318" y2="73.9648" width="0.3048" layer="1"/>
+<wire x1="4.318" y1="73.9648" x2="4.318" y2="80.899" width="0.3048" layer="1"/>
 <wire x1="4.318" y1="80.899" x2="3.497" y2="81.72" width="0.3048" layer="1"/>
 <wire x1="2.3462" y1="81.72" x2="3.497" y2="81.72" width="0.3048" layer="1"/>
